File: eagle/zero-tiny-ble.brd (EAGLE design)
At the start: 20 x 47 mm, 16 parts, among them U1 MAX1555, U2 attiny85, U3 HM-10

Commit message: updated silk screen.
Parts:
- renumbered LED-CHG to CHARGE, LED-CON to CONNECT
Routing:
- net 3.3V: track 123.1 -> 131.4 mm
Other:
- board text added: "By Zero Engineering www.zeroengineering.io"
- board text added: "Zero Tiny BLE V2.0"
- board text removed: "By Zero Engineering"
- board text removed: "Zero Tiny85 V2.0"
Changed lines of the file:
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@@
 <setting verticaltext="up"/>
 </settings>
-<grid distance="0.05" unitdist="inch" unit="inch" style="lines" multiple="1" display="no" altdistance="0.025" altunitdist="inch" altunit="inch"/>
+<grid distance="0.025" unitdist="inch" unit="inch" style="lines" multiple="1" display="no" altdistance="0.025" altunitdist="inch" altunit="inch"/>
 <layers>
 <layer number="1" name="Top" color="4" fill="1" visible="yes" active="yes"/>
@@
 <wire x1="19.99" y1="45.71" x2="0" y2="45.71" width="0" layer="20"/>
 <wire x1="0" y1="45.71" x2="0" y2="-1.27" width="0" layer="20"/>
-<text x="3.81" y="12.7" size="1.27" layer="121" font="fixed" rot="R90">Zero Tiny85 V2.0</text>
-<text x="19.05" y="11.43" size="1.27" layer="121" font="fixed" rot="R90">By Zero Engineering</text>
-<text x="3.81" y="41.91" size="0.6096" layer="121" rot="R90">GD</text>
-<text x="6.35" y="41.91" size="0.6096" layer="121" rot="R90">P5</text>
-<text x="8.89" y="41.91" size="0.6096" layer="121" rot="R90">P2</text>
-<text x="11.43" y="41.91" size="0.6096" layer="121" rot="R90">P1</text>
-<text x="13.97" y="41.91" size="0.6096" layer="121" rot="R90">P0</text>
-<text x="16.51" y="41.91" size="0.6096" layer="121" rot="R90">3.3</text>
+<text x="3.81" y="12.7" size="1.27" layer="121" font="fixed" rot="R90">Zero Tiny BLE V2.0</text>
+<text x="19.05" y="10.795" size="1.27" layer="121" font="fixed" rot="R90">By Zero Engineering
+www.zeroengineering.io</text>
+<text x="4.445" y="42.545" size="0.8128" layer="121" rot="R180">GD</text>
+<text x="6.985" y="42.545" size="0.8128" layer="121" rot="R180">P5</text>
+<text x="9.525" y="42.545" size="0.8128" layer="121" rot="R180">P2</text>
+<text x="12.065" y="42.545" size="0.8128" layer="121" rot="R180">P1</text>
+<text x="13.335" y="42.545" size="0.8128" layer="122" rot="MR180">P0</text>
+<text x="17.145" y="42.545" size="0.8128" layer="121" rot="R180">3.3</text>
 <text x="1.27" y="30.48" size="1.778" layer="121">*</text>
+<text x="15.875" y="42.545" size="0.8128" layer="122" rot="MR180">3.3</text>
+<text x="14.605" y="42.545" size="0.8128" layer="121" rot="R180">P0</text>
+<text x="8.255" y="42.545" size="0.8128" layer="122" rot="MR180">P2</text>
+<text x="10.795" y="42.545" size="0.8128" layer="122" rot="MR180">P1</text>
+<text x="5.715" y="42.545" size="0.8128" layer="122" rot="MR180">P5</text>
+<text x="3.175" y="42.545" size="0.8128" layer="122" rot="MR180">GD</text>
 </plain>
 <attributes>
@@
 </autorouter>
 <elements>
-<element name="C1" library="SparkFun-Capacitors" package="0805" value="1uF" x="8.89" y="24.13" rot="R270">
+<element name="C1" library="SparkFun-Capacitors" package="0805" value="1uF" x="8.89" y="24.13" smashed="yes" rot="R270">
 <attribute name="PROD_ID" value="CAP-08064" x="8.89" y="24.13" size="1.778" layer="27" rot="R270" display="off"/>
-</element>
-<element name="C2" library="SparkFun-Capacitors" package="0805" value="2.2uF" x="13.97" y="24.13" rot="R90">
+<attribute name="NAME" x="9.7155" y="24.892" size="0.4064" layer="25" rot="R270"/>
+<attribute name="VALUE" x="7.493" y="25.146" size="0.6096" layer="27" rot="R270"/>
+</element>
+<element name="C2" library="SparkFun-Capacitors" package="0805" value="2.2uF" x="13.97" y="24.13" smashed="yes" rot="R90">
 <attribute name="PROD_ID" value="CAP-11624" x="13.97" y="24.13" size="1.778" layer="27" rot="R90" display="off"/>
+<attribute name="NAME" x="13.1445" y="23.368" size="0.6096" layer="25" rot="R90"/>
+<attribute name="VALUE" x="15.367" y="23.114" size="0.6096" layer="27" rot="R90"/>
 </element>
 <element name="BAT-3.7V" library="adafruit" package="JST-PH-2-THM" value="" x="16.51" y="36.83" smashed="yes" rot="R270">
 <attribute name="NAME" x="13.01" y="39.63" size="0.8128" layer="25" font="vector" rot="R270"/>
 </element>
-<element name="LED-CON" library="adafruit" package="CHIPLED_0805" value="BLU" x="17.78" y="10.16" smashed="yes" rot="R270">
-<attribute name="NAME" x="16.51" y="8.89" size="0.6096" layer="25"/>
+<element name="CONNECT" library="adafruit" package="CHIPLED_0805" value="BLU" x="17.78" y="10.16" smashed="yes" rot="R270">
+<attribute name="NAME" x="12.065" y="9.525" size="0.6096" layer="25"/>
 <attribute name="VALUE" x="17.78" y="11.43" size="0.6096" layer="27"/>
 </element>
-<element name="R1" library="SparkFun-Resistors" package="0805" value="470R" x="10.16" y="19.05" rot="R90">
+<element name="R1" library="SparkFun-Resistors" package="0805" value="470R" x="10.16" y="19.05" smashed="yes" rot="R90">
 <attribute name="PROD_ID" value="RES-11622" x="10.16" y="19.05" size="1.778" layer="27" rot="R90" display="off"/>
-</element>
-<element name="R2" library="SparkFun-Resistors" package="0805" value="470R" x="13.97" y="19.05" rot="R270">
+<attribute name="NAME" x="9.3345" y="18.288" size="0.6096" layer="25" rot="R90"/>
+<attribute name="VALUE" x="11.557" y="18.034" size="0.6096" layer="27" rot="R90"/>
+</element>
+<element name="R2" library="SparkFun-Resistors" package="0805" value="470R" x="13.97" y="19.05" smashed="yes" rot="R270">
 <attribute name="PROD_ID" value="RES-11622" x="13.97" y="19.05" size="1.778" layer="27" rot="R270" display="off"/>
+<attribute name="NAME" x="14.7955" y="19.812" size="0.6096" layer="25" rot="R270"/>
+<attribute name="VALUE" x="12.573" y="20.066" size="0.6096" layer="27" rot="R270"/>
 </element>
 <element name="U$2" library="LP2985" package="SOT25" value="LP2985AIM5-3.3" x="12.7" y="12.7" smashed="yes">
@@
 <element name="U1" library="SparkFun-PowerIC" package="SOT23-5" value="MAX1555" x="7.62" y="12.7"/>
 <element name="JP1" library="SparkFun-Connectors" package="USB-MINIB-NOSTOP" value="USB-SMD-NS" x="10.16" y="3.81" rot="R90"/>
-<element name="LED-CHG" library="adafruit" package="CHIPLED_0805" value="GRN" x="2.54" y="10.16" smashed="yes" rot="R270">
-<attribute name="NAME" x="0" y="8.89" size="0.6096" layer="25"/>
+<element name="CHARGE" library="adafruit" package="CHIPLED_0805" value="GRN" x="2.54" y="10.16" smashed="yes" rot="R270">
+<attribute name="NAME" x="4.445" y="9.525" size="0.6096" layer="25"/>
 <attribute name="VALUE" x="2.54" y="11.43" size="0.6096" layer="27"/>
 </element>
-<element name="R3" library="SparkFun-Resistors" package="0805" value="470R" x="6.35" y="19.05" rot="R90">
+<element name="R3" library="SparkFun-Resistors" package="0805" value="470R" x="6.35" y="19.05" smashed="yes" rot="R90">
 <attribute name="PROD_ID" value="RES-11622" x="6.35" y="19.05" size="1.778" layer="27" rot="R90" display="off"/>
-</element>
-<element name="C4" library="SparkFun-Capacitors" package="0805" value="1uF" x="6.35" y="24.13" rot="R270">
+<attribute name="NAME" x="5.5245" y="18.288" size="0.6096" layer="25" rot="R90"/>
+<attribute name="VALUE" x="7.747" y="18.034" size="0.6096" layer="27" rot="R90"/>
+</element>
+<element name="C4" library="SparkFun-Capacitors" package="0805" value="1uF" x="6.35" y="24.13" smashed="yes" rot="R270">
 <attribute name="PROD_ID" value="CAP-08064" x="6.35" y="24.13" size="1.778" layer="27" rot="R270" display="off"/>
-</element>
-<element name="C3" library="SparkFun-Passives" package="0805" value="10nF" x="11.43" y="24.13" rot="R270"/>
+<attribute name="NAME" x="7.1755" y="24.892" size="0.4064" layer="25" rot="R270"/>
+<attribute name="VALUE" x="4.953" y="25.146" size="0.6096" layer="27" rot="R270"/>
+</element>
+<element name="C3" library="SparkFun-Passives" package="0805" value="10nF" x="11.43" y="24.13" smashed="yes" rot="R270">
+<attribute name="NAME" x="12.2555" y="24.892" size="0.6096" layer="25" rot="R270"/>
+<attribute name="VALUE" x="10.033" y="25.146" size="0.6096" layer="27" rot="R270"/>
+</element>
 <element name="JP2" library="SparkFun-Connectors" package="1X06" value="" x="3.81" y="44.45">
 <attribute name="PROD_ID" value="CONN-08437" x="3.81" y="44.45" size="1.778" layer="27" display="off"/>
@@
 <contactref element="C2" pad="2"/>
 <contactref element="U2" pad="4"/>
-<contactref element="LED-CON" pad="C"/>
+<contactref element="CONNECT" pad="C"/>
 <contactref element="U1" pad="2"/>
 <contactref element="U3" pad="13"/>
@@
 <wire x1="18.7452" y1="10.287" x2="18.83" y2="10.16" width="0.254" layer="1"/>
 <wire x1="14.1732" y1="24.9174" x2="13.97" y2="25.03" width="0.254" layer="1"/>
+<wire x1="3.8862" y1="36.1188" x2="3.8862" y2="44.3484" width="0.254" layer="16"/>
 </signal>
 <signal name="VCC">
@@
 <signal name="N$16">
 <contactref element="R2" pad="2"/>
-<contactref element="LED-CON" pad="A"/>
+<contactref element="CONNECT" pad="A"/>
 <wire x1="14.1732" y1="15.5448" x2="14.1732" y2="18.0594" width="0.254" layer="1"/>
 <wire x1="16.6878" y1="13.0302" x2="14.1732" y2="15.5448" width="0.254" layer="1"/>
@@
 <signal name="N$3">
 <contactref element="U1" pad="3"/>
-<contactref element="LED-CHG" pad="C"/>
+<contactref element="CHARGE" pad="C"/>
 <wire x1="5.9436" y1="10.0584" x2="3.6576" y2="10.0584" width="0.254" layer="1"/>
 <wire x1="6.1722" y1="9.8298" x2="5.9436" y2="10.0584" width="0.254" layer="1"/>
@@
 <signal name="N$1">
 <contactref element="R3" pad="1"/>
-<contactref element="LED-CHG" pad="A"/>
+<contactref element="CHARGE" pad="A"/>
 <wire x1="1.6002" y1="13.4874" x2="1.6002" y2="10.287" width="0.254" layer="1"/>
 <wire x1="6.1722" y1="18.0594" x2="1.6002" y2="13.4874" width="0.254" layer="1"/>
@@
 </board>
 </drawing>
+<compatibility>
+<note version="6.3" minversion="6.2.2" severity="warning">
+Since Version 6.2.2 text objects can contain more than one line,
+which will not be processed correctly with this version.
+</note>
+</compatibility>
 </eagle>
