File: eagle/zero-tiny-ble.sch (EAGLE design)
At the start: 16 parts, among them U1 MAX1555, U2 attiny85, U3 HM-10

Commit message: updated silk screen.
Parts:
- renumbered LED-CHG to CHARGE, LED-CON to CONNECT
Changed lines of the file:
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@@
 <grid distance="0.01" unitdist="inch" unit="inch" style="lines" multiple="1" display="no" altdistance="0.01" altunitdist="inch" altunit="inch"/>
 <layers>
-<layer number="1" name="Top" color="4" fill="1" visible="yes" active="no"/>
-<layer number="16" name="Bottom" color="1" fill="1" visible="yes" active="no"/>
-<layer number="17" name="Pads" color="2" fill="1" visible="yes" active="no"/>
-<layer number="18" name="Vias" color="2" fill="1" visible="yes" active="no"/>
-<layer number="19" name="Unrouted" color="6" fill="1" visible="yes" active="no"/>
-<layer number="20" name="Dimension" color="15" fill="1" visible="yes" active="no"/>
-<layer number="21" name="tPlace" color="7" fill="1" visible="yes" active="no"/>
-<layer number="22" name="bPlace" color="7" fill="1" visible="yes" active="no"/>
-<layer number="23" name="tOrigins" color="15" fill="1" visible="yes" active="no"/>
-<layer number="24" name="bOrigins" color="15" fill="1" visible="yes" active="no"/>
-<layer number="25" name="tNames" color="7" fill="1" visible="yes" active="no"/>
-<layer number="26" name="bNames" color="7" fill="1" visible="yes" active="no"/>
-<layer number="27" name="tValues" color="7" fill="1" visible="yes" active="no"/>
-<layer number="28" name="bValues" color="7" fill="1" visible="yes" active="no"/>
+<layer number="1" name="Top" color="4" fill="1" visible="no" active="no"/>
+<layer number="16" name="Bottom" color="1" fill="1" visible="no" active="no"/>
+<layer number="17" name="Pads" color="2" fill="1" visible="no" active="no"/>
+<layer number="18" name="Vias" color="2" fill="1" visible="no" active="no"/>
+<layer number="19" name="Unrouted" color="6" fill="1" visible="no" active="no"/>
+<layer number="20" name="Dimension" color="15" fill="1" visible="no" active="no"/>
+<layer number="21" name="tPlace" color="7" fill="1" visible="no" active="no"/>
+<layer number="22" name="bPlace" color="7" fill="1" visible="no" active="no"/>
+<layer number="23" name="tOrigins" color="15" fill="1" visible="no" active="no"/>
+<layer number="24" name="bOrigins" color="15" fill="1" visible="no" active="no"/>
+<layer number="25" name="tNames" color="7" fill="1" visible="no" active="no"/>
+<layer number="26" name="bNames" color="7" fill="1" visible="no" active="no"/>
+<layer number="27" name="tValues" color="7" fill="1" visible="no" active="no"/>
+<layer number="28" name="bValues" color="7" fill="1" visible="no" active="no"/>
 <layer number="29" name="tStop" color="7" fill="3" visible="no" active="no"/>
 <layer number="30" name="bStop" color="7" fill="6" visible="no" active="no"/>
@@
 <layer number="35" name="tGlue" color="7" fill="4" visible="no" active="no"/>
 <layer number="36" name="bGlue" color="7" fill="5" visible="no" active="no"/>
-<layer number="37" name="tTest" color="7" fill="1" visible="yes" active="no"/>
-<layer number="38" name="bTest" color="7" fill="1" visible="yes" active="no"/>
+<layer number="37" name="tTest" color="7" fill="1" visible="no" active="no"/>
+<layer number="38" name="bTest" color="7" fill="1" visible="no" active="no"/>
 <layer number="39" name="tKeepout" color="4" fill="11" visible="no" active="no"/>
 <layer number="40" name="bKeepout" color="1" fill="11" visible="no" active="no"/>
@@
 <layer number="44" name="Drills" color="7" fill="1" visible="no" active="no"/>
 <layer number="45" name="Holes" color="7" fill="1" visible="no" active="no"/>
-<layer number="46" name="Milling" color="3" fill="1" visible="yes" active="no"/>
-<layer number="47" name="Measures" color="7" fill="1" visible="yes" active="no"/>
-<layer number="48" name="Document" color="7" fill="1" visible="yes" active="no"/>
-<layer number="49" name="Reference" color="7" fill="1" visible="yes" active="no"/>
-<layer number="50" name="dxf" color="7" fill="1" visible="yes" active="no"/>
-<layer number="51" name="tDocu" color="7" fill="1" visible="yes" active="no"/>
-<layer number="52" name="bDocu" color="7" fill="1" visible="yes" active="no"/>
-<layer number="53" name="tGND_GNDA" color="7" fill="9" visible="yes" active="no"/>
-<layer number="54" name="bGND_GNDA" color="1" fill="9" visible="yes" active="no"/>
-<layer number="56" name="wert" color="7" fill="1" visible="yes" active="no"/>
-<layer number="57" name="tCAD" color="7" fill="1" visible="yes" active="no"/>
+<layer number="46" name="Milling" color="3" fill="1" visible="no" active="no"/>
+<layer number="47" name="Measures" color="7" fill="1" visible="no" active="no"/>
+<layer number="48" name="Document" color="7" fill="1" visible="no" active="no"/>
+<layer number="49" name="Reference" color="7" fill="1" visible="no" active="no"/>
+<layer number="50" name="dxf" color="7" fill="1" visible="no" active="no"/>
+<layer number="51" name="tDocu" color="7" fill="1" visible="no" active="no"/>
+<layer number="52" name="bDocu" color="7" fill="1" visible="no" active="no"/>
+<layer number="53" name="tGND_GNDA" color="7" fill="9" visible="no" active="no"/>
+<layer number="54" name="bGND_GNDA" color="1" fill="9" visible="no" active="no"/>
+<layer number="56" name="wert" color="7" fill="1" visible="no" active="no"/>
+<layer number="57" name="tCAD" color="7" fill="1" visible="no" active="no"/>
 <layer number="90" name="Modules" color="5" fill="1" visible="yes" active="yes"/>
 <layer number="91" name="Nets" color="2" fill="1" visible="yes" active="yes"/>
@@
 <part name="R2" library="SparkFun-Resistors" deviceset="0.3OHM-1/8W-1%(0805)" device="" value="470R"/>
 <part name="GND10" library="SparkFun-Aesthetics" deviceset="GND2" device=""/>
-<part name="LED-CON" library="adafruit" deviceset="LED" device="CHIPLED_0805" value="BLU"/>
+<part name="CONNECT" library="adafruit" deviceset="LED" device="CHIPLED_0805" value="BLU"/>
 <part name="U1" library="SparkFun-PowerIC" deviceset="MAX1555" device=""/>
 <part name="JP1" library="SparkFun-Connectors" deviceset="USB" device="-SMD-NS"/>
@@
 <part name="GND1" library="SparkFun-Aesthetics" deviceset="GND2" device=""/>
 <part name="GND7" library="SparkFun-Aesthetics" deviceset="GND2" device=""/>
-<part name="LED-CHG" library="adafruit" deviceset="LED" device="CHIPLED_0805" value="GRN"/>
+<part name="CHARGE" library="adafruit" deviceset="LED" device="CHIPLED_0805" value="GRN"/>
 <part name="R3" library="SparkFun-Resistors" deviceset="0.3OHM-1/8W-1%(0805)" device="" value="470R"/>
 <part name="GND8" library="SparkFun-Aesthetics" deviceset="GND2" device=""/>
@@
 <instance part="R2" gate="G$1" x="209.55" y="133.35"/>
 <instance part="GND10" gate="G$1" x="232.41" y="133.35" rot="R90"/>
-<instance part="LED-CON" gate="G$1" x="219.71" y="133.35" rot="R90"/>
+<instance part="CONNECT" gate="G$1" x="219.71" y="133.35" rot="R90"/>
 <instance part="U1" gate="G$1" x="81.28" y="27.94"/>
 <instance part="JP1" gate="G$1" x="35.56" y="33.02" rot="R180"/>
@@
 <instance part="GND1" gate="G$1" x="177.8" y="102.87"/>
 <instance part="GND7" gate="G$1" x="44.45" y="43.18" rot="R180"/>
-<instance part="LED-CHG" gate="G$1" x="74.93" y="12.7" rot="R270"/>
+<instance part="CHARGE" gate="G$1" x="74.93" y="12.7" rot="R270"/>
 <instance part="R3" gate="G$1" x="87.63" y="12.7"/>
 <instance part="GND8" gate="G$1" x="55.88" y="59.69"/>
@@
 </segment>
 <segment>
-<pinref part="LED-CON" gate="G$1" pin="C"/>
+<pinref part="CONNECT" gate="G$1" pin="C"/>
 <pinref part="GND10" gate="G$1" pin="3.3V"/>
 <wire x1="224.79" y1="133.35" x2="229.87" y2="133.35" width="0.1524" layer="91"/>
@@
 <segment>
 <pinref part="R2" gate="G$1" pin="2"/>
-<pinref part="LED-CON" gate="G$1" pin="A"/>
+<pinref part="CONNECT" gate="G$1" pin="A"/>
 <wire x1="214.63" y1="133.35" x2="217.17" y2="133.35" width="0.1524" layer="91"/>
 </segment>
@@
 <wire x1="66.04" y1="25.4" x2="66.04" y2="12.7" width="0.1524" layer="91"/>
 <wire x1="66.04" y1="12.7" x2="69.85" y2="12.7" width="0.1524" layer="91"/>
-<pinref part="LED-CHG" gate="G$1" pin="C"/>
+<pinref part="CHARGE" gate="G$1" pin="C"/>
 </segment>
 </net>
@@
 <segment>
 <pinref part="R3" gate="G$1" pin="1"/>
-<pinref part="LED-CHG" gate="G$1" pin="A"/>
+<pinref part="CHARGE" gate="G$1" pin="A"/>
 <wire x1="77.47" y1="12.7" x2="82.55" y2="12.7" width="0.1524" layer="91"/>
 </segment>
